File: KICAD/CAN-Relay-Board.kicad_pcb (KiCad board)
At the start: 2 copper layers, 38.1 x 30.5 mm, 28 parts, among them J1 UPDI Header, J2 Conn_01x04_Female, J3 UART Header, U1 AZ1117-5.0, U2 MCP2551-I-SN, U3 ATtiny414-SS, U5 MCP2515-xSO, Y1 8MHz

Commit message: Schematic 90% complete
Parts:
- added D2: NRVA4007T3G, Diode_SMD:D_SMA, F.Cu at (184.9, 104.6)
- added D3: NRVA4007T3G, Diode_SMD:D_SMA, F.Cu at (191.0, 122.9)
- added D4: NRVA4007T3G, Diode_SMD:D_SMA, F.Cu at (185.4, 85.1)
- added K1: CP1SA-12V-X, eec:Panasonic-CP1SA-12V-X-MFG, F.Cu at (203.3, 87.9)
- added K2: CP1SA-12V-X, eec:Panasonic-CP1SA-12V-X-MFG, F.Cu at (203.3, 122.9)
- added K3: CP1SA-12V-X, eec:Panasonic-CP1SA-12V-X-MFG, F.Cu at (203.2, 105.4)
- added K4: CP1SA-12V-X, eec:Panasonic-CP1SA-12V-X-MFG, F.Cu at (203.2, 140.7)
- added Q1: MMBT2222A-TP, Package_TO_SOT_SMD:SOT-23, F.Cu at (189.7, 110.7)
- added Q2: MMBT2222A-TP, Package_TO_SOT_SMD:SOT-23, F.Cu at (189.5, 102.1)
- added Q3: MMBT2222A-TP, Package_TO_SOT_SMD:SOT-23, F.Cu at (190.0, 96.3)
- added Q4: MMBT2222A-TP, Package_TO_SOT_SMD:SOT-23, F.Cu at (190.4, 82.1)
- added R10: 1K, Resistor_SMD:R_0603_1608Metric_Pad0.98x0.95mm_HandSolder, F.Cu at (189.8, 89.2)
- added R8: 1K, Resistor_SMD:R_0603_1608Metric_Pad0.98x0.95mm_HandSolder, F.Cu at (190.2, 85.6)
- added R9: 1K, Resistor_SMD:R_0603_1608Metric_Pad0.98x0.95mm_HandSolder, F.Cu at (189.8, 91.7)
- added U4: 1-2834011-3, 1-2834011-3:CONN_1-2834011-3, F.Cu at (217.5, 94.0)
- added U6: 1-2834011-3, 1-2834011-3:CONN_1-2834011-3, F.Cu at (217.4, 122.9)
- added U7: 1-2834011-3, 1-2834011-3:CONN_1-2834011-3, F.Cu at (217.4, 108.4)
- added U8: 1-2834011-3, 1-2834011-3:CONN_1-2834011-3, F.Cu at (217.7, 137.1)
- D1: value LED -> NRVA4007T3G; footprint LED_SMD:LED_0603_1608Metric_Pad1.05x0.95mm_HandSolder -> Diode_SMD:D_SMA
- R6: value 150 -> 1K
- moved U2 92.6 mm to (157.0, 109.2)
- moved D1 88.2 mm to (190.8, 142.7), turned to 90 degrees
- moved R1 86.9 mm to (176.4, 84.0)
- moved R4 86.9 mm to (176.4, 85.5)
- moved U5 86.5 mm to (168.1, 89.2)
- moved C5 86.3 mm to (158.5, 87.4)
- moved Y1 86.3 mm to (158.1, 91.5)
- moved C6 86.3 mm to (163.6, 95.2)
- moved R2 86.3 mm to (167.4, 96.8)
- moved C4 86.3 mm to (158.2, 95.2)
- moved C1 85.1 mm to (173.2, 140.1)
- moved U1 85.1 mm to (178.1, 142.6)
- moved C2 85.1 mm to (182.9, 140.1)
- moved R6 83.9 mm to (189.6, 105.9)
- moved R3 81.9 mm to (161.5, 113.8)
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Connections:
- net /Analog renamed /RELAY_4
- D1 pad 1: Net-(D1-Pad1) -> VCC
- D1 pad 2: unconnected-(D1-Pad2) -> Net-(D1-Pad2)
- R6 pad 1: GND -> /RELAY_1
- R6 pad 2: Net-(D1-Pad1) -> Net-(Q1-Pad1)
- U3 pad 2: unconnected-(U3-Pad2) -> /RELAY_2
- U3 pad 3: unconnected-(U3-Pad3) -> /RELAY_3
- U3 pad 8: unconnected-(U3-Pad8) -> /RELAY_1
Routing:
- net +5V: track 102.5 -> 0.00 mm, vias 3 -> 0
- net VCC: track 50.6 -> 0.00 mm, vias 1 -> 0
- net /UPDI: track 29.3 -> 0.00 mm
- net Net-(U2-Pad1): track 27.9 -> 0.00 mm, vias 2 -> 0
- net Net-(U2-Pad4): track 24.2 -> 0.00 mm, vias 2 -> 0
- net unconnected-(D1-Pad2): track 22.2 -> 0.00 mm
- net /RESET: track 21.0 -> 0.00 mm, vias 2 -> 0
- net /CS: track 18.7 -> 0.00 mm
- net Net-(R2-Pad1): track 17.9 -> 0.00 mm, vias 2 -> 0
- net Net-(C5-Pad1): track 13.5 -> 0.00 mm
- net /CAN_L: track 12.4 -> 0.00 mm
- net /INT: track 11.9 -> 0.00 mm, vias 2 -> 0
- net /MOSI: track 11.5 -> 0.00 mm, vias 2 -> 0
- net Net-(R3-Pad2): track 11.4 -> 0.00 mm, vias 2 -> 0
- net /CAN_H: track 11.4 -> 0.00 mm
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Other:
- board size 38.1 x 30.5 mm -> 84.1 x 75.4 mm
